File: ProMicroKeypad.kicad_sch (KiCad schematic)
At the start: 0 parts

Commit message: Components added
Parts:
- added R? (x9): R_US, symbol Device:R_US
- added SW?: RotaryEncoder_Switch, symbol Device:RotaryEncoder_Switch
- added U? (x9): CherryMX_LED, symbol CherryMX:CherryMX_LED
- added U?: ProMicro, symbol promicro:ProMicro
Other:
- title: (none) -> Arduino ProMicro Shortcut Keypad
