File: ProMicroKeypad.kicad_sch (KiCad schematic)
At the start: 20 parts

Commit message: Finished component placement and annotation
Parts:
- R1, R2, R3, R4, R5, R6, R7, R8, R9: renamed from R?; value R_US -> 150R
- gave numbers to parts that had none: 11
Connections:
- net LedC1: now reaches R4.1
- net LedC1: now also R1.1, R7.1, U10. (VCC)
- net at R4.2: now also U4.3 (K)
- net LedC2: now reaches R5.1
- net LedC2: now also R2.1, R8.1, U10. (VCC)
- net at R5.2: now also U5.3 (K)
- net SwC1: now reaches U7.1
- net SwC1: now also U1.1, U10. (VCC), U4.1
- net SwR3: now reaches U7.2
- net SwR3: now also U10. (VCC), U8.2, U9.2
- net at U7.3 (K): now also R7.2
- net LedR3: now reaches U7.4 (A)
- net LedR3: now also U10. (VCC), U8.4 (A), U9.4 (A)
- net SwC2: now reaches U5.1
- net SwC2: now also U10. (VCC), U2.1, U8.1
- net SwR2: now reaches U5.2
- net SwR2: now also U10. (VCC), U4.2, U6.2
- net LedR2: now reaches U5.4 (A)
- net LedR2: now also U10. (VCC), U4.4 (A), U6.4 (A)
- net at R1.2: now also U1.3 (K)
- net SwC3: now reaches U9.1
- net SwC3: now also U3.1, U6.1
- net at U9.3 (K): now also R9.2
- net SwR1: now reaches U2.2
- net SwR1: now also U1.2, U10. (VCC), U3.2
- net at U2.3 (K): now also R2.2
- net LedR1: now reaches U2.4 (A)
- net LedR1: now also U1.4 (A), U10. (VCC), U3.4 (A)
- net LedC3: now reaches R6.1
- net LedC3: now also R3.1, R9.1, U10. (VCC)
- net at R6.2: now also U6.3 (K)
- net EncA: now reaches SW1.A
- net EncA: now also U10. (VCC)
- net EncB: now reaches SW1.B
- net EncB: now also U10. (VCC)
- net GND: now reaches SW1.C
- net GND: now also SW1.S2, U10. (VCC)
- net EncSw: now reaches SW1.S1
- net EncSw: now also U10. (VCC)
- net at U8.3 (K): now also R8.2
- net at R3.2: now also U3.3 (K)
- no-connect marks 0 -> 8
Other:
- note added: "Arduino Pro-Micro (Leonardo)"
- note added: "Cherry MX keys with LED"
- note added: "LED resistors = 150R R = (5 - 2) / 0.02"
- note added: "Rotary encoder w/ swtich"
- moved on the sheet: R1, R2, R3, R4, R5, R6, R7, R8, R9, SW1, U1, U10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

Commit message: Footprints assigned
Parts:
- R1, R2, R3, R4, R5, R6, R7, R8, R9: footprint (none) -> Resistor_SMD:R_1206_3216Metric_Pad1.30x1.75mm_HandSolder
- SW1: footprint (none) -> Rotary_Encoder:RotaryEncoder_Alps_EC11E-Switch_Vertical_H20mm
- U1, U2, U3, U4, U5, U6, U7, U8, U9: footprint (none) -> Cherry MX Full:CherryMX_1.00u_PCB_LED
- U10: footprint (none) -> promicro:ProMicro

Commit message: PCB design done
Connections:
- net EncA: now also U10.18 (F6); no longer U10. (VCC)
- net EncB: now also U10.19 (F5); no longer U10. (VCC)
- net EncSw: now also U10.17 (F7); no longer U10. (VCC)
- net GND: now also U10.3 (GND); no longer U10. (VCC)
- net LedC1: now also U10.14 (B2); no longer U10. (VCC)
- net LedC2: now also U10.15 (B3); no longer U10. (VCC)
- net LedC3: now also U10.16 (B1); no longer U10. (VCC)
- net LedR1: now also U10.11 (B4); no longer U10. (VCC)
- net LedR2: now also U10.12 (B5); no longer U10. (VCC)
- net LedR3: now also U10.13 (B6); no longer U10. (VCC)
- net SwC1: now also U10.8 (C6); no longer U10. (VCC)
- net SwC2: now also U10.9 (D7); no longer U10. (VCC)
- net SwR1: now also U10.5 (SCL); no longer U10. (VCC)
- net SwR2: now also U10.6 (SDA); no longer U10. (VCC)
- net SwR3: now also U10.10 (E6), U10.7 (D4); no longer U10. (VCC)
Changed lines of the file:
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@@
       (effects (font (size 1.524 1.524)))
     )
-    (pin "")
-    (pin "")
-    (pin "")
-    (pin "")
-    (pin "")
-    (pin "")
-    (pin "")
-    (pin "")
-    (pin "")
-    (pin "")
-    (pin "")
-    (pin "")
-    (pin "")
-    (pin "")
-    (pin "")
-    (pin "")
-    (pin "")
-    (pin "")
-    (pin "")
-    (pin "")
-    (pin "")
-    (pin "")
-    (pin "")
-    (pin "")
+    (pin "1")
+    (pin "10")
+    (pin "11")
+    (pin "12")
+    (pin "13")
+    (pin "14")
+    (pin "15")
+    (pin "16")
+    (pin "17")
+    (pin "18")
+    (pin "19")
+    (pin "2")
+    (pin "20")
+    (pin "21")
+    (pin "22")
+    (pin "23")
+    (pin "24")
+    (pin "3")
+    (pin "4")
+    (pin "5")
+    (pin "6")
+    (pin "7")
+    (pin "8")
+    (pin "9")
   )
   (sheet_instances

Commit message: Fixing schematic and PCB
Connections:
- net SwC3: now also U10.10 (E6)
- net SwR3: no longer U10.10 (E6)
Changed lines of the file:
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@@
     (effects (font (size 1.27 1.27)) (justify left bottom))
   )
-  (label "SwR3" (at 204.47 69.85 0)
+  (label "SwC3" (at 204.47 69.85 0)
     (effects (font (size 1.27 1.27)) (justify left bottom))
   )
@@
     (pin "2")
   )
-  (symbol (lib_id "CherryMX:CherryMX_LED") (at 55.88 40.64 0) (unit 1)
+  (symbol (lib_name "CherryMX:CherryMX_LED_1") (lib_id "CherryMX:CherryMX_LED") (at 55.88 40.64 0) (unit 1)
     (in_bom yes) (on_board yes) (fields_autoplaced)
     (property "Reference" "U1" (id 0) (at 55.88 33.02 0))
@@
     (pin "4")
   )
-  (symbol (lib_id "CherryMX:CherryMX_LED") (at 55.88 58.42 0) (unit 1)
+  (symbol (lib_name "CherryMX:CherryMX_LED_4") (lib_id "CherryMX:CherryMX_LED") (at 55.88 58.42 0) (unit 1)
     (in_bom yes) (on_board yes) (fields_autoplaced)
     (property "Reference" "U4" (id 0) (at 55.88 50.8 0))
@@
     (pin "4")
   )
-  (symbol (lib_id "CherryMX:CherryMX_LED") (at 55.88 76.2 0) (unit 1)
+  (symbol (lib_name "CherryMX:CherryMX_LED_7") (lib_id "CherryMX:CherryMX_LED") (at 55.88 76.2 0) (unit 1)
     (in_bom yes) (on_board yes) (fields_autoplaced)
     (property "Reference" "U7" (id 0) (at 55.88 68.58 0))
@@
     (pin "4")
   )
-  (symbol (lib_id "CherryMX:CherryMX_LED") (at 92.71 40.64 0) (unit 1)
+  (symbol (lib_name "CherryMX:CherryMX_LED_2") (lib_id "CherryMX:CherryMX_LED") (at 92.71 40.64 0) (unit 1)
     (in_bom yes) (on_board yes) (fields_autoplaced)
     (property "Reference" "U2" (id 0) (at 92.71 33.02 0))
@@
     (pin "4")
   )
-  (symbol (lib_id "CherryMX:CherryMX_LED") (at 92.71 58.42 0) (unit 1)
+  (symbol (lib_name "CherryMX:CherryMX_LED_5") (lib_id "CherryMX:CherryMX_LED") (at 92.71 58.42 0) (unit 1)
     (in_bom yes) (on_board yes) (fields_autoplaced)
     (property "Reference" "U5" (id 0) (at 92.71 50.8 0))
@@
     (pin "4")
   )
-  (symbol (lib_id "CherryMX:CherryMX_LED") (at 92.71 76.2 0) (unit 1)
+  (symbol (lib_name "CherryMX:CherryMX_LED_8") (lib_id "CherryMX:CherryMX_LED") (at 92.71 76.2 0) (unit 1)
     (in_bom yes) (on_board yes) (fields_autoplaced)
     (property "Reference" "U8" (id 0) (at 92.71 68.58 0))
@@
     (pin "4")
   )
-  (symbol (lib_id "CherryMX:CherryMX_LED") (at 129.54 40.64 0) (unit 1)
+  (symbol (lib_name "CherryMX:CherryMX_LED_3") (lib_id "CherryMX:CherryMX_LED") (at 129.54 40.64 0) (unit 1)
     (in_bom yes) (on_board yes) (fields_autoplaced)
     (property "Reference" "U3" (id 0) (at 129.54 33.02 0))
@@
     (pin "4")
   )
-  (symbol (lib_id "CherryMX:CherryMX_LED") (at 129.54 58.42 0) (unit 1)
+  (symbol (lib_name "CherryMX:CherryMX_LED_6") (lib_id "CherryMX:CherryMX_LED") (at 129.54 58.42 0) (unit 1)
     (in_bom yes) (on_board yes) (fields_autoplaced)
     (property "Reference" "U6" (id 0) (at 129.54 50.8 0))
