File: ProMicroKeypad.kicad_pcb (KiCad board)
At the start: 0 parts

Commit message: PCB design done
Parts:
- added R1: 150R, Resistor_SMD:R_1206_3216Metric_Pad1.30x1.75mm_HandSolder, F.Cu at (127.0, 91.5)
- added R2: 150R, Resistor_SMD:R_1206_3216Metric_Pad1.30x1.75mm_HandSolder, F.Cu at (127.0, 85.0)
- added R3: 150R, Resistor_SMD:R_1206_3216Metric_Pad1.30x1.75mm_HandSolder, F.Cu at (127.0, 78.5)
- added R4: 150R, Resistor_SMD:R_1206_3216Metric_Pad1.30x1.75mm_HandSolder, F.Cu at (127.0, 72.0)
- added R5: 150R, Resistor_SMD:R_1206_3216Metric_Pad1.30x1.75mm_HandSolder, F.Cu at (127.0, 65.5)
- added R6: 150R, Resistor_SMD:R_1206_3216Metric_Pad1.30x1.75mm_HandSolder, F.Cu at (163.5, 58.0)
- added R7: 150R, Resistor_SMD:R_1206_3216Metric_Pad1.30x1.75mm_HandSolder, F.Cu at (163.5, 52.5)
- added R8: 150R, Resistor_SMD:R_1206_3216Metric_Pad1.30x1.75mm_HandSolder, F.Cu at (163.6, 47.0)
- added R9: 150R, Resistor_SMD:R_1206_3216Metric_Pad1.30x1.75mm_HandSolder, F.Cu at (163.5, 41.5)
- added SW1: RotaryEncoder_Switch, Rotary_Encoder:RotaryEncoder_Alps_EC11E-Switch_Vertical_H20mm, F.Cu at (172.2, 47.5)
- added U1: CherryMX_LED, Cherry MX Full:CherryMX_1.00u_PCB_LED, F.Cu at (141.5, 92.0)
- added U10: ProMicro, promicro:ProMicro, F.Cu at (138.5, 49.0)
- added U2: CherryMX_LED, Cherry MX Full:CherryMX_1.00u_PCB_LED, F.Cu at (161.5, 92.0)
- added U3: CherryMX_LED, Cherry MX Full:CherryMX_1.00u_PCB_LED, F.Cu at (181.5, 92.0)
- added U4: CherryMX_LED, Cherry MX Full:CherryMX_1.00u_PCB_LED, F.Cu at (141.5, 71.5)
- added U5: CherryMX_LED, Cherry MX Full:CherryMX_1.00u_PCB_LED, F.Cu at (161.5, 71.5)
- added U6: CherryMX_LED, Cherry MX Full:CherryMX_1.00u_PCB_LED, F.Cu at (181.5, 71.5)
- added U7: CherryMX_LED, Cherry MX Full:CherryMX_1.00u_PCB_LED, F.Cu at (202.5, 51.0)
- added U8: CherryMX_LED, Cherry MX Full:CherryMX_1.00u_PCB_LED, F.Cu at (202.5, 71.5)
- added U9: CherryMX_LED, Cherry MX Full:CherryMX_1.00u_PCB_LED, F.Cu at (202.5, 92.0)
Routing:
- net /LedR3: track 0.00 -> 114.7 mm
- net /SwR3: track 0.00 -> 113.8 mm
- net /SwC1: track 0.00 -> 97.1 mm
- net Net-(R9-Pad2): track 0.00 -> 91.2 mm
- net /SwC2: track 0.00 -> 85.7 mm
- net /LedC3: track 0.00 -> 82.7 mm
- net /LedR1: track 0.00 -> 81.7 mm
- net /LedC1: track 0.00 -> 78.8 mm
- net GND: track 0.00 -> 75.5 mm
- net /SwR1: track 0.00 -> 74.9 mm
- net /LedC2: track 0.00 -> 72.5 mm
- net /LedR2: track 0.00 -> 68.0 mm
- net Net-(R3-Pad2): track 0.00 -> 59.4 mm
- net /SwR2: track 0.00 -> 58.4 mm
- net Net-(R8-Pad2): track 0.00 -> 53.7 mm
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Other:
- board outline added: 93 x 67 mm
- copper layers 0 -> 2
