File: ProMicroKeypad.kicad_pcb (KiCad board)
At the start: 2 copper layers, 93 x 67 mm, 20 parts, among them SW1 RotaryEncoder_Switch, U1 CherryMX_LED, U10 ProMicro, U2 CherryMX_LED, U3 CherryMX_LED, U4 CherryMX_LED, U5 CherryMX_LED, U6 CherryMX_LED, U7 CherryMX_LED, U8 CherryMX_LED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

Commit message: Board completed
Routing:
- added copper zone on B.Cu, net GND
Other:
- board text added: "ProMicro Keypad v1.0"

Commit message: Fixing schematic and PCB
Connections:
- U10 pad 1: unconnected-(U10-Pad1) -> (no net)
- U10 pad 10: /SwR3 -> /SwC3
- U10 pad 2: unconnected-(U10-Pad2) -> (no net)
- U10 pad 20: unconnected-(U10-Pad20) -> (no net)
- U10 pad 21: unconnected-(U10-Pad21) -> (no net)
- U10 pad 22: unconnected-(U10-Pad22) -> (no net)
- U10 pad 23: unconnected-(U10-Pad23) -> (no net)
- U10 pad 24: unconnected-(U10-Pad24) -> (no net)
- U10 pad 4: unconnected-(U10-Pad4) -> (no net)
Routing:
- net /SwC3: track 41.5 -> 84.6 mm
- net /SwR3: track 113.8 -> 115.5 mm
Other:
- board text added: "A(+) C(-)"
